File: Hardware/SparkFun_Qwiic_Directional_Pad.kicad_pcb (KiCad board)
At the start: 2 copper layers, 25.4 x 25.4 mm, 62 parts, among them J1 Qwiic_RA, J2 Conn_01x04, J3 Qwiic_RA, J5 I2C, SW2 Nav Switch, U4 PCA9557PW

Commit message: Fix page names.
Parts:
- added JP6: I²C, SparkFun-Jumper:Jumper_3_NC-2_Trace, B.Cu at (140.0, 110.5)
- added R13: 2.2k, SparkFun-Resistor:R_0603_1608Metric, B.Cu at (137.2, 111.4)
- added R7: 2.2k, SparkFun-Resistor:R_0603_1608Metric, B.Cu at (137.2, 109.5)
- added kibuzzard-66F182A6: G***, kibuzzard-66F182A6, B.Cu at (141.9, 110.5)
- G***: footprint SparkFun-Aesthetic:SparkFun_Logo_8mm -> SparkFun-Aesthetic:SparkFun_Logo_NoFlame_8mm
- moved Ref** 20.6 mm to (154.9, 93.7)
- moved G1 19.9 mm to (214.6, 168.3)
- moved G*** 15.9 mm to (156.5, 112.4), turned to 180 degrees
- moved G*** 7.16 mm to (143.1, 104.8), turned to -90 degrees
Routing:
- net SDA: track 45.6 -> 53.8 mm
- net SCL: track 49.4 -> 56.9 mm
- net Net-(JP6-A): track 0.00 -> 2.07 mm
- net Net-(JP6-B): track 0.00 -> 2.07 mm
- net 3.3V: track 68.0 -> 70.1 mm
- net GND: vias 11 -> 19
Other:
- board text added: "Finish: HASL"
- board text removed: "Controlled Impedance: JLC7628"
- board text removed: "Finish: ENIG"
- board text removed: "Inner Copper Weight: 0.5oz"
- board text removed: "Material: TG155"
- board text removed: "No Clean Process"
